File: KiCad/Par2Ser.kicad_pcb (KiCad board)
At the start: 4 copper layers, 47 x 50 mm, 36 parts, among them J1 DB25_Male, J2 USB_C_Receptacle_USB2.0, U1 LC4032V-5TN48C, U2 FT240XS-R

Commit message: Add JTAG header
Parts:
- added J3: Conn_02x05_Odd_Even, Connector_PinHeader_2.54mm:PinHeader_2x05_P2.54mm_Vertical, F.Cu at (127.7, 106.1)
- moved C2 2.00 mm to (134.7, 117.6)
- moved C6 2.00 mm to (136.7, 117.6), turned to 270 degrees
Routing:
- net TCK: track 25.4 -> 2.22 mm
- net TDI: track 23.1 -> 1.86 mm
- net VCC: track 12.9 -> 7.37 mm
- net TMS: track 24.4 -> 19.2 mm
- net TD0: track 15.8 -> 10.5 mm
Other:
- board text added: "3V3"
- board text added: "GND"
- board text added: "JTAG"
- board text added: "NC"
- board text added: "TCK"
- board text added: "TDI"
- board text added: "TDO"
- board text added: "TMS"
Changed lines of the file:
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@@
   (general
     (thickness 1.6)
-    (drawings 31)
-    (tracks 513)
+    (drawings 42)
+    (tracks 509)
     (zones 0)
-    (modules 36)
-    (nets 78)
+    (modules 37)
+    (nets 82)
   )
   (page A4)
@@
   (net 76 "Net-(R9-Pad1)")
   (net 77 "Net-(R10-Pad1)")
+  (net 78 "Net-(J3-Pad10)")
+  (net 79 "Net-(J3-Pad9)")
+  (net 80 "Net-(J3-Pad8)")
+  (net 81 TDO)
   (net_class Default "This is the default net class."
     (clearance 0.1524)
@@
     (add_net "Net-(J2-PadA8)")
     (add_net "Net-(J2-PadB8)")
+    (add_net "Net-(J3-Pad10)")
+    (add_net "Net-(J3-Pad8)")
+    (add_net "Net-(J3-Pad9)")
     (add_net "Net-(R10-Pad1)")
     (add_net "Net-(R9-Pad1)")
@@
     (add_net TD0)
     (add_net TDI)
+    (add_net TDO)
     (add_net TMS)
     (add_net TXE)
@@
     (add_net VCC)
     (add_net WR)
+  )
+  (module Connector_PinHeader_2.54mm:PinHeader_2x05_P2.54mm_Vertical (layer F.Cu)
+    (at 127.71 106.11)
+    (descr "Through hole straight pin header, 2x05, 2.54mm pitch, double rows")
+    (tags "Through hole pin header THT 2x05 2.54mm double row")
+    (fp_text reference J3 (at 1.27 -2.33) (layer F.SilkS) hide
+      (effects (font (size 1 1) (thickness 0.15)))
+    )
+    (fp_text value Conn_02x05_Odd_Even (at 1.27 12.49) (layer F.Fab) hide
+      (effects (font (size 1 1) (thickness 0.15)))
+    )
+    (fp_text user %R (at 1.27 5.08 90) (layer F.Fab) hide
+      (effects (font (size 1 1) (thickness 0.15)))
+    )
+    (fp_line (start 0 -1.27) (end 3.81 -1.27) (layer F.Fab) (width 0.1))
+    (fp_line (start 3.81 -1.27) (end 3.81 11.43) (layer F.Fab) (width 0.1))
+    (fp_line (start 3.81 11.43) (end -1.27 11.43) (layer F.Fab) (width 0.1))
+    (fp_line (start -1.27 11.43) (end -1.27 0) (layer F.Fab) (width 0.1))
+    (fp_line (start -1.27 0) (end 0 -1.27) (layer F.Fab) (width 0.1))
+    (fp_line (start -1.8 -1.8) (end -1.8 11.95) (layer F.CrtYd) (width 0.05))
+    (fp_line (start -1.8 11.95) (end 4.35 11.95) (layer F.CrtYd) (width 0.05))
+    (fp_line (start 4.35 11.95) (end 4.35 -1.8) (layer F.CrtYd) (width 0.05))
+    (fp_line (start 4.35 -1.8) (end -1.8 -1.8) (layer F.CrtYd) (width 0.05))
+    (pad 10 thru_hole oval (at 2.54 10.16) (size 1.7 1.7) (drill 0.8) (layers *.Cu *.Mask)
+      (net 78 "Net-(J3-Pad10)"))
+    (pad 9 thru_hole oval (at 0 10.16) (size 1.7 1.7) (drill 0.8) (layers *.Cu *.Mask)
+      (net 79 "Net-(J3-Pad9)"))
+    (pad 8 thru_hole oval (at 2.54 7.62) (size 1.7 1.7) (drill 0.8) (layers *.Cu *.Mask)
+      (net 80 "Net-(J3-Pad8)"))
+    (pad 7 thru_hole oval (at 0 7.62) (size 1.7 1.7) (drill 0.8) (layers *.Cu *.Mask)
+      (net 81 TDO))
+    (pad 6 thru_hole oval (at 2.54 5.08) (size 1.7 1.7) (drill 0.8) (layers *.Cu *.Mask)
+      (net 16 3V3))
+    (pad 5 thru_hole oval (at 0 5.08) (size 1.7 1.7) (drill 0.8) (layers *.Cu *.Mask)
+      (net 32 TDI))
+    (pad 4 thru_hole oval (at 2.54 2.54) (size 1.7 1.7) (drill 0.8) (layers *.Cu *.Mask)
+      (net 1 GND))
+    (pad 3 thru_hole oval (at 0 2.54) (size 1.7 1.7) (drill 0.8) (layers *.Cu *.Mask)
+      (net 34 TMS))
+    (pad 2 thru_hole oval (at 2.54 0) (size 1.7 1.7) (drill 0.8) (layers *.Cu *.Mask)
+      (net 1 GND))
+    (pad 1 thru_hole rect (at 0 0) (size 1.7 1.7) (drill 0.8) (layers *.Cu *.Mask)
+      (net 33 TCK))
   )
   (module Capacitor_SMD:C_0603_1608Metric_Pad1.08x0.95mm_HandSolder (layer F.Cu)
@@
   )
   (module Capacitor_SMD:C_0805_2012Metric_Pad1.18x1.45mm_HandSolder (layer F.Cu)
-    (at 132.7 117.6 90)
+    (at 134.7 117.6 90)
     (descr "Capacitor SMD 0805 (2012 Metric), square (rectangular) end terminal, IPC_7351 nominal with elongated pad for handsoldering. (Body size source: IPC-SM-782 page 76, https://www.pcb-3d.com/wordpress/wp-content/uploads/ipc-sm-782a_amendment_1_and_2.pdf, https://docs.google.com/spreadsheets/d/1BsfQQcO9C6DZCsRaXUlFlo91Tg2WpOkGARC1WS5S8t0/edit?usp=sharing), generated with kicad-footprint-generator")
     (tags "capacitor handsolder")
@@
   )
   (module Capacitor_SMD:C_0805_2012Metric_Pad1.18x1.45mm_HandSolder (layer F.Cu)
-    (at 134.7 117.6 90)
+    (at 136.7 117.6 270)
     (descr "Capacitor SMD 0805 (2012 Metric), square (rectangular) end terminal, IPC_7351 nominal with elongated pad for handsoldering. (Body size source: IPC-SM-782 page 76, https://www.pcb-3d.com/wordpress/wp-content/uploads/ipc-sm-782a_amendment_1_and_2.pdf, https://docs.google.com/spreadsheets/d/1BsfQQcO9C6DZCsRaXUlFlo91Tg2WpOkGARC1WS5S8t0/edit?usp=sharing), generated with kicad-footprint-generator")
     (tags "capacitor handsolder")
     (attr smd)
-    (fp_text reference C6 (at 2.6 0.2 180) (layer F.SilkS)
+    (fp_text reference C6 (at -2.6 -0.2 180) (layer F.SilkS)
       (effects (font (size 1 1) (thickness 0.15)))
     )
@@
       (effects (font (size 0.5 0.5) (thickness 0.08)))
     )
-    (pad 2 smd roundrect (at 1.0375 0 90) (size 1.175 1.45) (layers F.Cu F.Paste F.Mask) (roundrect_rratio 0.2127659574468085)
-      (net 1 GND))
-    (pad 1 smd roundrect (at -1.0375 0 90) (size 1.175 1.45) (layers F.Cu F.Paste F.Mask) (roundrect_rratio 0.213)
+    (pad 2 smd roundrect (at 1.0375 0 270) (size 1.175 1.45) (layers F.Cu F.Paste F.Mask) (roundrect_rratio 0.2127659574468085)
+      (net 1 GND))
+    (pad 1 smd roundrect (at -1.0375 0 270) (size 1.175 1.45) (layers F.Cu F.Paste F.Mask) (roundrect_rratio 0.213)
       (net 21 VCC) (zone_connect 2))
     (model ${KISYS3DMOD}/Capacitor_SMD.3dshapes/C_0805_2012Metric.wrl
@@
       (rotate (xyz 90 180 180))
     )
+  )
+  (gr_text JTAG (at 128.85 118.9) (layer F.SilkS)
+    (effects (font (size 1.2 1.2) (thickness 0.15)))
+  )
+  (gr_text GND (at 132.25 104.8 90) (layer F.SilkS)
+    (effects (font (size 1 1) (thickness 0.15)))
+  )
+  (gr_text GND (at 132.25 108.3 90) (layer F.SilkS)
+    (effects (font (size 1 1) (thickness 0.15)))
+  )
+  (gr_text 3V3 (at 132.25 111.65 90) (layer F.SilkS)
+    (effects (font (size 1 1) (thickness 0.15)))
+  )
+  (gr_text NC (at 132.25 114.65 90) (layer F.SilkS)
+    (effects (font (size 1 1) (thickness 0.15)))
+  )
+  (gr_text NC (at 132.25 117.9 90) (layer F.SilkS)
+    (effects (font (size 1 1) (thickness 0.15)))
+  )
+  (gr_text NC (at 125.5 117.9 90) (layer F.SilkS)
+    (effects (font (size 1 1) (thickness 0.15)))
+  )
+  (gr_text TCK (at 125.5 104.8 90) (layer F.SilkS)
+    (effects (font (size 1 1) (thickness 0.15)))
+  )
+  (gr_text TMS (at 125.5 108.3 90) (layer F.SilkS)
+    (effects (font (size 1 1) (thickness 0.15)))
+  )
+  (gr_text TDI (at 125.5 111.4 90) (layer F.SilkS)
+    (effects (font (size 1 1) (thickness 0.15)))
+  )
+  (gr_text TDO (at 125.5 114.65 90) (layer F.SilkS)
+    (effects (font (size 1 1) (thickness 0.15)))
   )
   (gr_text AMIGAAAAA (at 168 105.5 90) (layer F.SilkS)
@@
   (segment (start 167.5 110.8) (end 167.5 112) (width 0.5) (layer F.Cu) (net 16))
   (segment (start 167.5 110.8) (end 168.8 112.1) (width 0.5) (layer F.Cu) (net 16))
-  (segment (start 132.7 118.6375) (end 132.7 122.275) (width 0.8) (layer F.Cu) (net 21))
-  (segment (start 132.7 118.6375) (end 134.7 118.6375) (width 0.8) (layer F.Cu) (net 21))
-  (segment (start 134.7 118.6375) (end 135.6625 118.6375) (width 0.8) (layer F.Cu) (net 21))
-  (segment (start 135.6625 118.6375) (end 136.8 117.5) (width 0.8) (layer F.Cu) (net 21))
-  (segment (start 136.8 117.5) (end 136.8 112.8) (width 0.8) (layer F.Cu) (net 21))
+  (segment (start 132.7 120.6375) (end 134.7 118.6375) (width 0.8) (layer F.Cu) (net 21))
+  (segment (start 132.7 122.275) (end 132.7 120.6375) (width 0.8) (layer F.Cu) (net 21))
+  (segment (start 136.7 116.6) (end 136.7 116.5625) (width 0.8) (layer F.Cu) (net 21))
+  (segment (start 134.7 118.6) (end 136.7 116.6) (width 0.8) (layer F.Cu) (net 21))
+  (segment (start 134.7 118.6375) (end 134.7 118.6) (width 0.8) (layer F.Cu) (net 21))
   (segment (start 164.12 87.254) (end 164.12 93) (width 0.4) (layer F.Cu) (net 22))
   (segment (start 140.22 127.2) (end 140.78 127.2) (width 0.3) (layer F.Cu) (net 24))
@@
   (segment (start 148.05 114.439087) (end 148.631371 115.020458) (width 0.25) (layer F.Cu) (net 32))
   (segment (start 148.05 113.4) (end 148.05 114.439087) (width 0.25) (layer F.Cu) (net 32))
-  (segment (start 148.05 113.4) (end 126.8 113.4) (width 0.25) (layer B.Cu) (net 32))
   (via (at 150.4 111.2) (size 0.8) (drill 0.4) (layers F.Cu B.Cu) (net 33))
   (segment (start 151.481982 110.800001) (end 152.166905 111.484924) (width 0.25) (layer F.Cu) (net 33))
   (segment (start 150.799999 110.800001) (end 151.481982 110.800001) (width 0.25) (layer F.Cu) (net 33))
   (segment (start 150.4 111.2) (end 150.799999 110.800001) (width 0.25) (layer F.Cu) (net 33))
-  (segment (start 150.4 111.2) (end 127.2 111.2) (width 0.3) (layer B.Cu) (net 33))
   (via (at 145.5 103.5) (size 0.8) (drill 0.4) (layers F.Cu B.Cu) (net 34))
   (segment (start 145.5 104.110913) (end 146.368629 104.979542) (width 0.25) (layer F.Cu) (net 34))
   (segment (start 145.5 103.5) (end 145.5 104.110913) (width 0.25) (layer F.Cu) (net 34))
   (segment (start 138.86 99.5) (end 132.46 105.9) (width 0.25) (layer B.Cu) (net 34))
-  (segment (start 132.46 105.9) (end 127.2 105.9) (width 0.25) (layer B.Cu) (net 34))
   (segment (start 140.46 101.1) (end 143.1 101.1) (width 0.25) (layer B.Cu) (net 34))
   (segment (start 143.1 101.1) (end 145.5 103.5) (width 0.25) (layer B.Cu) (net 34))
@@
   (segment (start 142.833095 108.515076) (end 142.318019 108) (width 0.25) (layer F.Cu) (net 35))
   (segment (start 142.318019 108) (end 132.5 108) (width 0.25) (layer F.Cu) (net 35))
-  (segment (start 132.5 108) (end 127.25 108) (width 0.25) (layer F.Cu) (net 35))
   (segment (start 157.4925 114.6925) (end 157.4925 119.75) (width 0.25) (layer F.Cu) (net 36))
   (segment (start 156.1 113.3) (end 157.4925 114.6925) (width 0.25) (layer F.Cu) (net 36))
